Commit message: velodyne 3d test init.

File: cartographer_ros/urdf/velodyne_h.urdf (robot description, URDF)
Before this commit: robot cartographer_backpack_3d, 4 links, 3 joints
Joints:
- joint horizontal_vlp16_link_joint: origin xyz=0.01 0. 0.19 rpy=0. -0.1745 3.1416 -> xyz=0.15 0. 0.01 rpy=0. 0. 0.
- joint imu_link_joint: origin xyz=0 0 0 rpy=3.1416 0 0 -> xyz=0. 0. 0. rpy=0. 0. 0.
- joint vertical_vlp16_link_joint: origin xyz=0.19 0. 0.04 rpy=0. -1.3963 0. -> xyz=0.10 0. 0.15 rpy=0. -1.3963 0.

Commit message: work for 2 velodyne.

File: cartographer_ros/urdf/velodyne_h.urdf (robot description, URDF)
Before this commit: robot cartographer_backpack_3d, 4 links, 3 joints
Joints:
- joint horizontal_vlp16_link_joint: origin xyz=0.15 0. 0.01 rpy=0. 0. 0. -> xyz=0.155 0. 0.020 rpy=0. 0. 0.034906584
- joint vertical_vlp16_link_joint: origin xyz=0.10 0. 0.15 rpy=0. -1.3963 0. -> xyz=0.115 0. 0.160 rpy=0. 0.78539815 -0.069813169
